Commit message: now two links can move

File: ROS/src/manip/urdf/manip.urdf (robot description, URDF)
Before this commit: robot manip, 4 links, 3 joints
Joints:
- joint joint_2: axis 0 0 0 -> 0 1 0; limit lower=0 upper=0 effort=0 velocity=0 -> lower=-3.14 upper=3.14 effort=100 velocity=0.1; origin xyz=0 0 0 rpy=0 0 0 -> xyz=0 0 0.19 rpy=0 0 0
